File: Hardware/Dash/ConnectorPCB/ConnectorPCB/ConnectorPCB.kicad_sch (KiCad schematic)
At the start: 3 parts, among them J1 776276-1, J2 2.54mm 1x4, J3 2.54mm 1x4

Commit message: PCB R0.1.0
Connections:
- net CAN_H: now also J1.6, J3.4; no longer J1.4, J2.4
- net GND: now also J1.4, J2.4; no longer J1.6, J3.4
Changed lines of the file:
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@@
     (stroke (width 0) (type default))
   )
-  (wire (pts (xy 63.5 76.835) (xy 78.74 76.835))
+  (wire (pts (xy 49.53 76.835) (xy 78.74 76.835))
+    (stroke (width 0) (type default))
+  )
+  (wire (pts (xy 136.525 76.835) (xy 142.24 76.835))
     (stroke (width 0) (type default))
   )
@@
     (stroke (width 0) (type default))
   )
-  (wire (pts (xy 136.525 65.405) (xy 142.24 65.405))
+  (wire (pts (xy 124.46 65.405) (xy 124.46 66.675))
+    (stroke (width 0) (type default))
+  )
+  (wire (pts (xy 142.24 65.405) (xy 124.46 65.405))
     (stroke (width 0) (type default))
   )
@@
     (stroke (width 0) (type default))
   )
-  (wire (pts (xy 60.96 62.865) (xy 66.675 62.865))
-    (stroke (width 0) (type default))
-  )
-  (wire (pts (xy 63.5 67.945) (xy 63.5 76.835))
-    (stroke (width 0) (type default))
-  )
-  (wire (pts (xy 142.24 76.835) (xy 135.89 76.835))
+  (wire (pts (xy 49.53 62.865) (xy 49.53 76.835))
+    (stroke (width 0) (type default))
+  )
+  (wire (pts (xy 49.53 62.865) (xy 66.675 62.865))
     (stroke (width 0) (type default))
   )
@@
     (stroke (width 0) (type default))
   )
+  (wire (pts (xy 60.96 67.945) (xy 66.675 67.945))
+    (stroke (width 0) (type default))
+  )
   (wire (pts (xy 60.96 60.325) (xy 66.675 60.325))
     (stroke (width 0) (type default))
@@
     (stroke (width 0) (type default))
   )
-  (wire (pts (xy 135.89 76.835) (xy 135.89 78.105))
-    (stroke (width 0) (type default))
-  )
   (wire (pts (xy 89.535 57.785) (xy 95.25 57.785))
     (stroke (width 0) (type default))
@@
     (stroke (width 0) (type default))
   )
-  (wire (pts (xy 66.675 67.945) (xy 63.5 67.945))
-    (stroke (width 0) (type default))
-  )
   (wire (pts (xy 136.525 69.215) (xy 142.24 69.215))
     (stroke (width 0) (type default))
@@
     (stroke (width 0) (type default))
   )
-  (global_label "CAN_H" (shape input) (at 60.96 62.865 180) (fields_autoplaced)
-    (effects (font (size 1.27 1.27)) (justify right))
-    (property "Intersheetrefs" "${INTERSHEET_REFS}" (at 52.067 62.865 0)
+  (global_label "CAN_H" (shape input) (at 60.96 67.945 180) (fields_autoplaced)
+    (effects (font (size 1.27 1.27)) (justify right))
+    (property "Intersheetrefs" "${INTERSHEET_REFS}" (at 52.067 67.945 0)
       (effects (font (size 1.27 1.27)) (justify right) hide)
     )
@@
     )
   )
-  (global_label "CAN_H" (shape input) (at 136.525 65.405 180) (fields_autoplaced)
-    (effects (font (size 1.27 1.27)) (justify right))
-    (property "Intersheetrefs" "${INTERSHEET_REFS}" (at 127.632 65.405 0)
+  (global_label "CAN_H" (shape input) (at 136.525 76.835 180) (fields_autoplaced)
+    (effects (font (size 1.27 1.27)) (justify right))
+    (property "Intersheetrefs" "${INTERSHEET_REFS}" (at 127.632 76.835 0)
       (effects (font (size 1.27 1.27)) (justify right) hide)
     )
@@
     )
   )
-  (symbol (lib_id "power:GND") (at 135.89 78.105 0) (unit 1)
+  (symbol (lib_id "power:GND") (at 124.46 66.675 0) (unit 1)
     (in_bom yes) (on_board yes) (dnp no) (fields_autoplaced)
-    (property "Reference" "#PWR02" (at 135.89 84.455 0)
-      (effects (font (size 1.27 1.27)) hide)
-    )
-    (property "Value" "GND" (at 135.89 83.185 0)
-      (effects (font (size 1.27 1.27)))
-    )
-    (property "Footprint" "" (at 135.89 78.105 0)
-      (effects (font (size 1.27 1.27)) hide)
-    )
-    (property "Datasheet" "" (at 135.89 78.105 0)
-      (effects (font (size 1.27 1.27)) hide)
-    )
+    (property "Reference" "#PWR02" (at 124.46 73.025 0)
+      (effects (font (size 1.27 1.27)) hide)
+    )
+    (property "Value" "GND" (at 124.46 71.755 0)
+      (effects (font (size 1.27 1.27)))
+    )
+    (property "Footprint" "" (at 124.46 66.675 0)
+      (effects (font (size 1.27 1.27)) hide)
+    )
+    (property "Datasheet" "" (at 124.46 66.675 0)
+      (effects (font (size 1.27 1.27)) hide)
+    )
