File: Hardware/Dash/AdvDash_5_inch/AdvDash_5_inch.kicad_pcb (KiCad board)
At the start: 4 copper layers, 150.6 x 90 mm, 186 parts, among them IC1 RV-8803-C7, IC2 74HCT1G126GW,125, J1 1-1734839-0, J2 54104-4031, J3 USB4110-GF-A, J4 2.54mm 1x4, J5 UART0, J6 2.54mm 1x4, J7 AUX, Q1 BSS139H6327XTSA1, Q2 AO3401A, Q3 S8050, SW1 RESET, SW2 RESET, T1 IRFR5305, U1 ESP32-S3-WROOM-1, U10 PC817, U2 TPS54331DDA, U3 MT9201, U4 USBLC6-2P6, U5 SN65HVD230, U6 BMP280, U7 CAT24C51, U8 LD1086DT33TR, U9 PC817

Commit message: PCB R0.1.0
Parts:
- H1, H2, H3, H4: footprint MountingHole:MountingHole_3.2mm_M3_Pad_Via -> MountingHole:MountingHole_3.2mm_M3_DIN965_Pad_TopBottom
- moved kibuzzard-653B3D6F 63.5 mm to (103.6, 110.5), turned to 90 degrees
- moved J7 54.9 mm to (148.3, 56.2)
- moved H2 8.86 mm to (83.5, 49.1)
- moved H1 8.43 mm to (211.3, 49.2)
- moved H3 6.23 mm to (82.7, 124.3)
- moved H4 6.13 mm to (211.7, 124.3)
- moved kibuzzard-653B4099 2.51 mm to (202.3, 53.7)
- moved kibuzzard-653B40B3 2.44 mm to (210.4, 53.7)
- moved SW1 2.33 mm to (202.3, 59.1)
- moved SW2 2.33 mm to (210.3, 59.1)
Routing:
- net /MCU/GPIO18: track 50.0 -> 19.1 mm
- net /MCU/GPIO17: track 44.9 -> 26.3 mm
- net GND: track 315.1 -> 323.9 mm, vias 141 -> 152
- net /MCU/GPIO42: track 27.6 -> 35.3 mm, vias 0 -> 2
- net /Display/DCLK: track 79.0 -> 76.8 mm
- net /Display/TP_RST: track 145.0 -> 142.8 mm
- net /Connector/SW_12V: track 15.8 -> 17.2 mm
- net +3.3V: track 109.8 -> 110.2 mm, vias 23 -> 27
Other:
- board size 150.6 x 90 mm -> 150.6 x 89.9 mm

Commit message: :adhesive_bandage: Minor change to the PCB
Parts:
- R10, R11, R12, R17, R24, R26, R27, R7: value 10k -> 10K
- R6: value 0 -> 0R

Commit message: :bug: PCB R0.2.0 Ready, change log in kicad files
Parts:
- removed J7: AUX, Connector_PinHeader_2.54mm:PinHeader_1x04_P2.54mm_Vertical_SMD_Pin1Left
- removed Q1: BSS139H6327XTSA1, PCM_Package_TO_SOT_SMD_AKL:SOT-23
- removed R11: 10K, Resistor_SMD:R_0805_2012Metric_Pad1.20x1.40mm_HandSolder
- added H5: MountingHole_Pad, MountingHole:MountingHole_2.2mm_M2_Pad, F.Cu at (130.2, 72.2)
- added H6: MountingHole_Pad, MountingHole:MountingHole_2.2mm_M2_Pad, F.Cu at (130.2, 101.8)
- added H7: MountingHole_Pad, MountingHole:MountingHole_2.2mm_M2_Pad, F.Cu at (169.0, 101.8)
- added IC3: 74HCT1G126GW,125, Package_TO_SOT_SMD:SOT-353_SC-70-5_Handsoldering, F.Cu at (212.2, 118.5)
- added JP4: ACT +/-, Jumper:SolderJumper-3_P1.3mm_Open_Pad1.0x1.5mm, F.Cu at (185.7, 56.2)
- added JP5: Reset Control, Jumper:SolderJumper-3_P1.3mm_Open_Pad1.0x1.5mm, F.Cu at (149.8, 56.5)
- added JP6: ACT +/-, Jumper:SolderJumper-3_P1.3mm_Open_Pad1.0x1.5mm, F.Cu at (185.8, 59.8)
- D13, D14, D15, D16, D17, D18, D19, D20, D21, D22, D23, D24, D25, D26, D27, D28, D29, D30: value WS2812B -> SK9822; footprint LED_SMD:LED_WS2812B_PLCC4_5.0x5.0mm_P3.2mm -> LED_SMD:LED_RGB_5050-6
- R10: value 10K -> 0R
- R3: value 332 -> 332k
- U1: value ESP32-S3-WROOM-1 -> ESP32-S3-WROOM-1-N4R8
- moved C44 3.34 mm to (213.2, 108.5)
- moved D13 3.07 mm to (217.0, 110.7), turned to 90 degrees
- moved D30 2.94 mm to (77.0, 110.8), turned to -90 degrees
- moved C33 2.77 mm to (80.8, 78.0)
- moved C45 2.32 mm to (213.2, 74.2)
- moved D15 2.32 mm to (217.0, 75.9), turned to 90 degrees
- moved C31 2.26 mm to (80.8, 113.0)
- moved D28 2.07 mm to (77.0, 75.8), turned to -90 degrees
- moved C34 2.02 mm to (80.8, 60.8)
- moved D16 1.55 mm to (216.9, 58.5), turned to 90 degrees
- moved D27 1.38 mm to (77.0, 58.5), turned to -90 degrees
- moved C47 1.25 mm to (213.2, 91.0)
- moved C46 1.03 mm to (213.3, 56.2)
- moved D14 0.82 mm to (217.0, 93.2), turned to 90 degrees
- moved C30 0.56 mm to (99.8, 49.0)
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Connections:
- D13 pad 1: +5V -> Net-(D13-DI)
- D13 pad 2: Net-(D13-DOUT) -> Net-(D13-CI)
- D13 pad 4: Net-(D13-DIN) -> +5V
- D14 pad 1: +5V -> Net-(D13-DO)
- D14 pad 2: Net-(D14-DOUT) -> Net-(D13-CO)
- D14 pad 4: Net-(D13-DOUT) -> +5V
- D15 pad 1: +5V -> Net-(D14-DO)
- D15 pad 2: Net-(D15-DOUT) -> Net-(D14-CO)
- D15 pad 4: Net-(D14-DOUT) -> +5V
- D16 pad 1: +5V -> Net-(D15-DO)
- D16 pad 2: Net-(D16-DOUT) -> Net-(D15-CO)
- D16 pad 4: Net-(D15-DOUT) -> +5V
- D17 pad 1: +5V -> Net-(D16-DO)
- D17 pad 2: Net-(D17-DOUT) -> Net-(D16-CO)
- D17 pad 4: Net-(D16-DOUT) -> +5V
- D18 pad 1: +5V -> Net-(D17-DO)
- D18 pad 2: Net-(D18-DOUT) -> Net-(D17-CO)
- D18 pad 4: Net-(D17-DOUT) -> +5V
- D19 pad 1: +5V -> Net-(D18-DO)
- D19 pad 2: Net-(D19-DOUT) -> Net-(D18-CO)
- D19 pad 4: Net-(D18-DOUT) -> +5V
- D20 pad 1: +5V -> Net-(D19-DO)
- D20 pad 2: Net-(D20-DOUT) -> Net-(D19-CO)
- D20 pad 4: Net-(D19-DOUT) -> +5V
- D21 pad 1: +5V -> Net-(D20-DO)
- D21 pad 2: Net-(D21-DOUT) -> Net-(D20-CO)
- D21 pad 4: Net-(D20-DOUT) -> +5V
- D22 pad 1: +5V -> Net-(D21-DO)
- D22 pad 2: Net-(D22-DOUT) -> Net-(D21-CO)
- D22 pad 4: Net-(D21-DOUT) -> +5V
- D23 pad 1: +5V -> Net-(D22-DO)
- D23 pad 2: Net-(D23-DOUT) -> Net-(D22-CO)
- D23 pad 4: Net-(D22-DOUT) -> +5V
- D24 pad 1: +5V -> Net-(D23-DO)
- D24 pad 2: Net-(D24-DOUT) -> Net-(D23-CO)
- D24 pad 4: Net-(D23-DOUT) -> +5V
- D25 pad 1: +5V -> Net-(D24-DO)
- D25 pad 2: Net-(D25-DOUT) -> Net-(D24-CO)
- D25 pad 4: Net-(D24-DOUT) -> +5V
- D26 pad 1: +5V -> Net-(D25-DO)
- D26 pad 2: Net-(D26-DOUT) -> Net-(D25-CO)
- D26 pad 4: Net-(D25-DOUT) -> +5V
- D27 pad 1: +5V -> Net-(D26-DO)
- D27 pad 2: Net-(D27-DOUT) -> Net-(D26-CO)
- D27 pad 4: Net-(D26-DOUT) -> +5V
- D28 pad 1: +5V -> Net-(D27-DO)
- D28 pad 2: Net-(D28-DOUT) -> Net-(D27-CO)
- D28 pad 4: Net-(D27-DOUT) -> +5V
- D29 pad 1: +5V -> Net-(D28-DO)
- D29 pad 2: Net-(D29-DOUT) -> Net-(D28-CO)
- D29 pad 4: Net-(D28-DOUT) -> +5V
- D30 pad 1: +5V -> Net-(D29-DO)
- D30 pad 2: unconnected-(D30-DOUT-Pad2) -> Net-(D29-CO)
- D30 pad 4: Net-(D29-DOUT) -> +5V
- IC2 pad 2: /LEDs/WLED_CRT -> /LEDs/WLED_CLK
- IC2 pad 4: Net-(D13-DIN) -> Net-(D13-CI)
- J1 pad 7: /Display/TP_RST -> Net-(JP5-C)
- Q3 pad 1: GND -> Net-(Q3-B)
- Q3 pad 2: Net-(Q3-B) -> GND
- R10 pad 1: Net-(Q1-D) -> /MCU/5V_EN
- U1 pad 10: /MCU/GPIO17 -> /MCU/5V_EN
- U1 pad 11: /MCU/GPIO18 -> /Display/TP_RST_2
- U1 pad 20: /Can Bus/CRX -> /LEDs/WLED_CLK
- U1 pad 21: /Can Bus/CTX -> /LEDs/WLED_CRT
- U1 pad 28: /SDA -> unconnected-(U1-SPIIO6/GPIO35/FSPID/SUBSPID-Pad28)
- U1 pad 29: /SCL -> unconnected-(U1-SPIIO7/GPIO36/FSPICLK/SUBSPICLK-Pad29)
- U1 pad 30: /MCU/5V_EN -> unconnected-(U1-SPIDQS/GPIO37/FSPIQ/SUBSPIQ-Pad30)
- U1 pad 31: /LEDs/WLED_CRT -> /SDA
- U1 pad 35: /MCU/GPIO42 -> /SCL
- U1 pad 36: /MCU/U0RXD -> Net-(JP6-C)
- U1 pad 37: /MCU/U0TXD -> Net-(JP4-C)
Routing:
- net Net-(JP5-C): track 0.00 -> 82.8 mm
- net /LEDs/WLED_CLK: track 0.00 -> 75.3 mm, vias 0 -> 2
- net /Display/TP_RST: track 142.8 -> 68.0 mm
- net /MCU/GPIO42: track 35.3 -> 0.00 mm, vias 2 -> 0
- net Net-(D26-DO): track 0.00 -> 31.3 mm
- net Net-(D16-DO): track 0.00 -> 30.7 mm
- net Net-(D26-DOUT): track 28.3 -> 0.00 mm
- net Net-(D16-DOUT): track 28.3 -> 0.00 mm
- net Net-(D16-CO): track 0.00 -> 27.8 mm
- net Net-(D26-CO): track 0.00 -> 27.8 mm
- net /MCU/GPIO17: track 26.3 -> 0.00 mm, vias 2 -> 0
- net /MCU/GPIO18: track 19.1 -> 0.00 mm, vias 2 -> 0
- net /MCU/5V_EN: track 126.6 -> 145.1 mm, vias 2 -> 1
- net Net-(D29-DOUT): track 16.7 -> 0.00 mm
- net Net-(D14-DOUT): track 16.6 -> 0.00 mm
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Other:
- outline, holes or cut-outs redrawn
- board text added: "R0.2.0 PCB - Desing by Daniel Gaviria"
- board text removed: "IO17"
- board text removed: "IO18"
- board text removed: "IO42"
- board text removed: "R0.1.0 PCB - Desing by Daniel Gaviria"
