File: Hardware/Dash/AdvDash_5_inch/AdvDash_5_inch.kicad_pcb (KiCad board)
At the start: 4 copper layers, 150.6 x 89.9 mm, 190 parts, among them IC1 RV-8803-C7, IC2 74HCT1G126GW,125, IC3 74HCT1G126GW,125, J1 1-1734839-0, J2 54104-4031, J3 USB4110-GF-A, J4 2.54mm 1x4, J5 UART0, J6 2.54mm 1x4, Q2 AO3401A, Q3 S8050, SW1 RESET, SW2 RESET, T1 IRFR5305, U1 ESP32-S3-WROOM-1-N4R8, U10 PC817, U2 TPS54331DDA, U3 MT9201, U4 USBLC6-2P6, U5 SN65HVD230, U6 BMP280, U7 CAT24C51, U8 LD1086DT33TR, U9 PC817

Commit message: 🚀 PCB R0.2.1
Parts:
- H5, H6, H7: footprint MountingHole:MountingHole_2.2mm_M2_Pad -> MountingHole:MountingHole_2.5mm_Pad
Other:
- board text added: "R0.2.1 PCB - Desing by Daniel Gaviria"
- board text removed: "R0.2.0 PCB - Desing by Daniel Gaviria"
