File: Hardware/Dash/AdvDash_5_inch/bmp280.kicad_sch (KiCad schematic)
At the start: 6 parts, among them U3 BMP280

Commit message: PCB R0.1.0
Other:
- company: (none) -> ADV.ECU - GNVPerformance
- title: (none) -> Barometric Pressure and Temperature

Commit message: :adhesive_bandage: Minor change to the PCB
Parts:
- C6, C7: LCSC (none) -> C15850
- D2: LCSC (none) -> C5345962
- R11, R7: value 10k -> 10K; LCSC (none) -> C17414
- U3: LCSC (none) -> C83291
Changed lines of the file:
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@@
+      (effects (font (size 1.27 1.27)) hide)
+    )
+    (property "LCSC" "C15850" (at 120.015 58.42 0)
       (effects (font (size 1.27 1.27)) hide)
     )
@@
       (effects (font (size 1.27 1.27)) hide)
     )
+    (property "LCSC" "C5345962" (at 90.805 68.58 0)
+      (effects (font (size 1.27 1.27)) hide)
+    )
     (pin "1")
     (pin "2")
@@
       (effects (font (size 1.27 1.27)) hide)
     )
+    (property "LCSC" "C15850" (at 127.635 58.42 0)
+      (effects (font (size 1.27 1.27)) hide)
+    )
     (pin "1")
     (pin "2")
@@
       (effects (font (size 1.27 1.27)))
     )
-    (property "Value" "10k" (at 83.185 57.15 0)
+    (property "Value" "10K" (at 83.185 57.15 0)
       (effects (font (size 1.27 1.27)) hide)
     )
@@
       (effects (font (size 1.27 1.27)) hide)
     )
+    (property "LCSC" "C17414" (at 86.995 55.88 0)
+      (effects (font (size 1.27 1.27)) hide)
+    )
     (pin "1")
     (pin "2")
@@
     )
     (property "Datasheet" "https://ae-bst.resource.bosch.com/media/_tech/media/datasheets/BST-BMP280-DS001.pdf" (at 106.045 66.04 0)
+      (effects (font (size 1.27 1.27)) hide)
+    )
+    (property "LCSC" "C83291" (at 106.045 66.04 0)
       (effects (font (size 1.27 1.27)) hide)
     )
@@
       (effects (font (size 1.27 1.27)))
     )
-    (property "Value" "10k" (at 85.725 57.15 0)
+    (property "Value" "10K" (at 85.725 57.15 0)
       (effects (font (size 1.27 1.27)) hide)
     )
@@
       (effects (font (size 1.27 1.27)) hide)
     )
+    (property "LCSC" "C17414" (at 89.535 55.88 0)
+      (effects (font (size 1.27 1.27)) hide)
+    )
