File: Hardware/Dash/AdvDash_5_inch/canbus.kicad_sch (KiCad schematic)
At the start: 7 parts, among them U10 SN65HVD230

Commit message: PCB R0.1.0
Other:
- company: (none) -> ADV.ECU - GNVPerformance
- title: (none) -> Can Bus Communication

Commit message: :adhesive_bandage: Minor change to the PCB
Parts:
- D1: LCSC (none) -> C5158054
- R32: value 10k -> 10K; LCSC (none) -> C17414
- R36: LCSC (none) -> C114245
- U10: LCSC (none) -> C12084
Changed lines of the file:
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@@
       (effects (font (size 1.27 1.27)))
     )
-    (property "Value" "10k" (at 85.09 69.85 0)
+    (property "Value" "10K" (at 85.09 69.85 0)
       (effects (font (size 1.27 1.27)))
     )
@@
     )
     (property "Datasheet" "~" (at 88.265 68.58 0)
+      (effects (font (size 1.27 1.27)) hide)
+    )
+    (property "LCSC" "C17414" (at 88.265 68.58 0)
       (effects (font (size 1.27 1.27)) hide)
     )
@@
       (effects (font (size 1.27 1.27)) hide)
     )
+    (property "LCSC" "C5158054" (at 117.475 68.58 0)
+      (effects (font (size 1.27 1.27)) hide)
+    )
     (pin "3")
     (pin "1")
@@
     )
     (property "Datasheet" "http://www.ti.com/lit/ds/symlink/sn65hvd230.pdf" (at 99.695 49.53 0)
+      (effects (font (size 1.27 1.27)) hide)
+    )
+    (property "LCSC" "C12084" (at 102.235 59.69 0)
       (effects (font (size 1.27 1.27)) hide)
     )
@@
       (effects (font (size 1.27 1.27)) hide)
     )
+    (property "LCSC" "C114245" (at 132.715 58.42 0)
+      (effects (font (size 1.27 1.27)) hide)
+    )

Commit message: 🚀 PCB R0.2.1
Parts:
- renumbered TP6 to TP10, TP6 to TP11
