File: Hardware/Dash/AdvDash_5_inch/connector.kicad_sch (KiCad schematic)
At the start: 2 parts, among them J4 2.54mm 1x4, J6 2.54mm 1x4

Commit message: PCB R0.1.0
Other:
- company: (none) -> ADV.ECU - GNVPerformance
- title: (none) -> Main Connector Interface

Commit message: :bug: PCB R0.2.0 Ready, change log in kicad files
Parts:
- added H5, H6, H7: MountingHole_Pad, MountingHole:MountingHole_2.2mm_M2_Pad, symbol Mechanical:MountingHole_Pad
Connections:
- net GND: now also H5.1, H6.1, H7.1
Other:
- note added: "Connector PCB MH"
- moved on the sheet: J4, J6

Commit message: 🚀 PCB R0.2.1
Parts:
- H5, H6, H7: footprint MountingHole:MountingHole_2.2mm_M2_Pad -> MountingHole:MountingHole_2.5mm_Pad
