File: Hardware/Dash/AdvDash_5_inch/eprom.kicad_sch (KiCad schematic)
At the start: 3 parts, among them U7 CAT24C51

Commit message: PCB R0.1.0
Other:
- company: (none) -> ADV.ECU - GNVPerformance
- title: (none) -> External Non-Volatile Memory

Commit message: :adhesive_bandage: Minor change to the PCB
Parts:
- C27: LCSC (none) -> C38141
- R29: LCSC (none) -> C149504
- U7: LCSC (none) -> C79986
Changed lines of the file:
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@@
+      (effects (font (size 1.27 1.27)) hide)
+    )
+    (property "LCSC" "C149504" (at 119.38 64.135 0)
       (effects (font (size 1.27 1.27)) hide)
     )
@@
       (effects (font (size 1.27 1.27)) hide)
     )
+    (property "LCSC" "C38141" (at 98.425 46.355 0)
+      (effects (font (size 1.27 1.27)) hide)
+    )
     (pin "1")
     (pin "2")
@@
       (effects (font (size 1.27 1.27)) hide)
     )
+    (property "LCSC" "C79986" (at 105.41 57.15 0)
+      (effects (font (size 1.27 1.27)) hide)
+    )

Commit message: 🚀 PCB R0.2.1
Parts:
- renumbered R29 to R31
