File: Hardware/Dash/AdvDash_5_inch/leds.kicad_sch (KiCad schematic)
At the start: 37 parts, among them IC2 74HCT1G126GW,125

Commit message: PCB R0.1.0
Other:
- company: (none) -> ADV.ECU - GNVPerformance
- title: (none) -> WS2812B RGB Leds

Commit message: :adhesive_bandage: Minor change to the PCB
Parts:
- C19: LCSC (none) -> C577419
- D13, D14, D15, D16, D17, D18, D19, D20, D21, D22, D23, D24, D25, D26, D27, D28, D29, D30: LCSC (none) -> C114586
- IC2: LCSC (none) -> C455064
Changed lines of the file:
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@@
       (effects (font (size 1.27 1.27)) (justify left top) hide)
+    )
+    (property "LCSC" "C114586" (at 190.5 118.745 0)
+      (effects (font (size 1.27 1.27)) hide)
     )
     (pin "1")
@@
       (effects (font (size 1.27 1.27)) hide)
     )
+    (property "LCSC" "C577419" (at 185.42 67.945 0)
+      (effects (font (size 1.27 1.27)) hide)
+    )
     (pin "1")
     (pin "2")
@@
       (effects (font (size 1.27 1.27)) (justify left top) hide)
     )
+    (property "LCSC" "C114586" (at 149.86 76.835 0)
+      (effects (font (size 1.27 1.27)) hide)
+    )
     (pin "1")
     (pin "2")
@@
       (effects (font (size 1.27 1.27)) (justify left top) hide)
     )
+    (property "LCSC" "C114586" (at 150.495 118.745 0)
+      (effects (font (size 1.27 1.27)) hide)
+    )
     (pin "1")
     (pin "2")
@@
       (effects (font (size 1.27 1.27)) hide)
     )
+    (property "LCSC" "C577419" (at 144.78 67.945 0)
+      (effects (font (size 1.27 1.27)) hide)
+    )
     (pin "1")
     (pin "2")
@@
       (effects (font (size 1.27 1.27)) (justify left top) hide)
     )
+    (property "LCSC" "C114586" (at 231.775 118.745 0)
+      (effects (font (size 1.27 1.27)) hide)
+    )
     (pin "1")
     (pin "2")
@@
       (effects (font (size 1.27 1.27)) hide)
     )
+    (property "LCSC" "C577419" (at 84.455 109.855 0)
+      (effects (font (size 1.27 1.27)) hide)
+    )
     (pin "1")
     (pin "2")
@@
       (effects (font (size 1.27 1.27)) hide)
     )
+    (property "LCSC" "C577419" (at 226.06 109.855 0)
+      (effects (font (size 1.27 1.27)) hide)
+    )
     (pin "1")
     (pin "2")
@@
     (property "Datasheet" "https://cdn-shop.adafruit.com/datasheets/WS2812B.pdf" (at 254 86.36 0)
       (effects (font (size 1.27 1.27)) (justify left top) hide)
+    )
+    (property "LCSC" "C114586" (at 251.46 76.835 0)
+      (effects (font (size 1.27 1.27)) hide)
     )
     (pin "1")
@@
       (effects (font (size 1.27 1.27)) hide)
     )
+    (property "LCSC" "C577419" (at 105.41 109.855 0)
+      (effects (font (size 1.27 1.27)) hide)
+    )
     (pin "1")
     (pin "2")
@@
     )
     (property "Datasheet" "~" (at 205.74 67.945 0)
+      (effects (font (size 1.27 1.27)) hide)
+    )
+    (property "LCSC" "C577419" (at 205.74 67.945 0)
       (effects (font (size 1.27 1.27)) hide)
     )
@@
       (effects (font (size 1.27 1.27)) (justify left top) hide)
     )
+    (property "LCSC" "C455064" (at 38.735 93.98 0)
+      (effects (font (size 1.27 1.27)) hide)
+    )
     (pin "1")
     (pin "2")
@@
       (effects (font (size 1.27 1.27)) (justify left top) hide)
     )
+    (property "LCSC" "C114586" (at 170.815 118.745 0)
+      (effects (font (size 1.27 1.27)) hide)
+    )
     (pin "1")
     (pin "2")
@@
       (effects (font (size 1.27 1.27)) hide)
     )
+    (property "LCSC" "C577419" (at 125.095 67.945 0)
+      (effects (font (size 1.27 1.27)) hide)
+    )
     (pin "1")
     (pin "2")
@@
       (effects (font (size 1.27 1.27)) hide)
     )
+    (property "LCSC" "C577419" (at 186.055 109.855 0)
+      (effects (font (size 1.27 1.27)) hide)
+    )
     (pin "1")
     (pin "2")
@@
       (effects (font (size 1.27 1.27)) hide)
     )
+    (property "LCSC" "C577419" (at 206.375 109.855 0)
+      (effects (font (size 1.27 1.27)) hide)
+    )
     (pin "1")
     (pin "2")
@@
       (effects (font (size 1.27 1.27)) hide)
     )
+    (property "LCSC" "C577419" (at 165.735 109.855 0)
+      (effects (font (size 1.27 1.27)) hide)
+    )
     (pin "1")
     (pin "2")
@@
       (effects (font (size 1.27 1.27)) (justify left top) hide)
     )
+    (property "LCSC" "C114586" (at 109.855 76.835 0)
+      (effects (font (size 1.27 1.27)) hide)
+    )
     (pin "1")
     (pin "2")
@@
       (effects (font (size 1.27 1.27)) (justify left top) hide)
     )
+    (property "LCSC" "C114586" (at 89.535 76.835 0)
+      (effects (font (size 1.27 1.27)) hide)
+    )
     (pin "1")
     (pin "2")
@@
       (effects (font (size 1.27 1.27)) (justify left top) hide)
     )
+    (property "LCSC" "C114586" (at 252.095 118.745 0)
+      (effects (font (size 1.27 1.27)) hide)
+    )
     (pin "1")
     (pin "2")
@@
       (effects (font (size 1.27 1.27)) (justify left top) hide)
     )
+    (property "LCSC" "C114586" (at 190.5 76.835 0)
+      (effects (font (size 1.27 1.27)) hide)
+    )
     (pin "1")
     (pin "2")
@@
       (effects (font (size 1.27 1.27)) hide)
     )
+    (property "LCSC" "C577419" (at 145.415 109.855 0)
+      (effects (font (size 1.27 1.27)) hide)
+    )
     (pin "1")
     (pin "2")
@@
       (effects (font (size 1.27 1.27)) (justify left top) hide)
     )
+    (property "LCSC" "C114586" (at 210.185 76.835 0)
+      (effects (font (size 1.27 1.27)) hide)
+    )
     (pin "1")
     (pin "2")
@@
       (effects (font (size 1.27 1.27)) (justify left top) hide)
     )
+    (property "LCSC" "C114586" (at 170.18 76.835 0)
+      (effects (font (size 1.27 1.27)) hide)
+    )
     (pin "1")
     (pin "2")
@@
       (effects (font (size 1.27 1.27)) hide)
     )
+    (property "LCSC" "C577419" (at 104.775 67.945 0)
+      (effects (font (size 1.27 1.27)) hide)
+    )
     (pin "1")
     (pin "2")
@@
       (effects (font (size 1.27 1.27)) (justify left top) hide)
     )
+    (property "LCSC" "C114586" (at 90.17 118.745 0)
+      (effects (font (size 1.27 1.27)) hide)
+    )
     (pin "1")
     (pin "2")
@@
       (effects (font (size 1.27 1.27)) hide)
     )
+    (property "LCSC" "C577419" (at 225.425 67.945 0)
+      (effects (font (size 1.27 1.27)) hide)
+    )
     (pin "1")
     (pin "2")
@@
       (effects (font (size 1.27 1.27)) hide)
     )
+    (property "LCSC" "C577419" (at 246.38 109.855 0)
+      (effects (font (size 1.27 1.27)) hide)
+    )
     (pin "1")
     (pin "2")
@@
       (effects (font (size 1.27 1.27)) hide)
     )
+    (property "LCSC" "C577419" (at 245.745 67.945 0)
+      (effects (font (size 1.27 1.27)) hide)
+    )
     (pin "1")
     (pin "2")
@@
       (effects (font (size 1.27 1.27)) hide)
     )
+    (property "LCSC" "C577419" (at 83.82 67.945 0)
+      (effects (font (size 1.27 1.27)) hide)
+    )
     (pin "1")
     (pin "2")
@@
     )
     (property "Datasheet" "~" (at 125.73 109.855 0)
+      (effects (font (size 1.27 1.27)) hide)
+    )
+    (property "LCSC" "C577419" (at 125.73 109.855 0)
       (effects (font (size 1.27 1.27)) hide)
     )
@@
       (effects (font (size 1.27 1.27)) hide)
     )
+    (property "LCSC" "C577419" (at 165.1 67.945 0)
+      (effects (font (size 1.27 1.27)) hide)
+    )
     (pin "1")
     (pin "2")
@@
       (effects (font (size 1.27 1.27)) (justify left top) hide)
     )
+    (property "LCSC" "C114586" (at 129.54 76.835 0)
+      (effects (font (size 1.27 1.27)) hide)
+    )
     (pin "1")
     (pin "2")
@@
       (effects (font (size 1.27 1.27)) (justify left top) hide)
     )
+    (property "LCSC" "C114586" (at 130.175 118.745 0)
+      (effects (font (size 1.27 1.27)) hide)
+    )
     (pin "1")
     (pin "2")
@@
     (property "Datasheet" "https://cdn-shop.adafruit.com/datasheets/WS2812B.pdf" (at 112.395 128.27 0)
       (effects (font (size 1.27 1.27)) (justify left top) hide)
+    )
+    (property "LCSC" "C114586" (at 109.855 118.745 0)
+      (effects (font (size 1.27 1.27)) hide)
     )
     (pin "1")
@@
       (effects (font (size 1.27 1.27)) (justify left top) hide)
     )
+    (property "LCSC" "C114586" (at 210.82 118.745 0)
+      (effects (font (size 1.27 1.27)) hide)
+    )
     (pin "1")
     (pin "2")
@@
       (effects (font (size 1.27 1.27)) (justify left top) hide)
     )
-    (pin "1")
+    (property "LCSC" "C114586" (at 230.505 76.835 0)
+      (effects (font (size 1.27 1.27)) hide)
+    )
+    (pin "1")

Commit message: :bug: PCB R0.2.0 Ready, change log in kicad files
Parts:
- added IC3: 74HCT1G126GW,125, Package_TO_SOT_SMD:SOT-353_SC-70-5_Handsoldering, symbol 74HCT1G126GW_125:74HCT1G126GW,125
- D13, D14, D15, D16, D17, D18, D19, D20, D21, D22, D23, D24, D25, D26, D27, D28, D29, D30: value WS2812B -> SK9822; footprint LED_SMD:LED_WS2812B_PLCC4_5.0x5.0mm_P3.2mm -> LED_SMD:LED_RGB_5050-6; symbol LED:WS2812B -> LED:APA102; LCSC C114586 -> C2829089
Connections:
- net +5V: now also D13.4 (VCC), D14.4 (VCC), D15.4 (VCC), D16.4 (VCC), D17.4 (VCC), D18.4 (VCC), D19.4 (VCC), D20.4 (VCC), D21.4 (VCC), D22.4 (VCC), D23.4 (VCC), D24.4 (VCC), D25.4 (VCC), D26.4 (VCC), D27.4 (VCC), D28.4 (VCC), D29.4 (VCC), D30.4 (VCC), IC3.1 (OE), IC3.5 (VCC); no longer D13.1 (VDD), D14.1 (VDD), D15.1 (VDD), D16.1 (VDD), D17.1 (VDD), D18.1 (VDD), D19.1 (VDD), D20.1 (VDD), D21.1 (VDD), D22.1 (VDD), D23.1 (VDD), D24.1 (VDD), D25.1 (VDD), D26.1 (VDD), D27.1 (VDD), D28.1 (VDD), D29.1 (VDD), D30.1 (VDD)
- net GND: now also IC3.3 (GND)
- net WLED_CRT: now also IC3.2 (A); no longer IC2.2 (A)
- net at D27.2 (CI): now also D26.5 (CO); no longer D28.4 (DIN)
- net at D26.2 (CI): now also D25.5 (CO); no longer D27.4 (DIN)
- net at D16.2 (CI): now also D15.5 (CO); no longer D17.4 (DIN)
- net at D15.2 (CI): now also D14.5 (CO); no longer D16.4 (DIN)
- net at D25.2 (CI): now also D24.5 (CO); no longer D26.4 (DIN)
- net at D24.2 (CI): now also D23.5 (CO); no longer D25.4 (DIN)
- net at D29.2 (CI): now also D28.5 (CO); no longer D30.4 (DIN)
- net at D28.2 (CI): now also D27.5 (CO); no longer D29.4 (DIN)
- net at D21.2 (CI): now also D20.5 (CO); no longer D22.4 (DIN)
- net at D20.2 (CI): now also D19.5 (CO); no longer D21.4 (DIN)
- net at IC2.4 (Y): now also D13.2 (CI); no longer D13.4 (DIN)
- net at D14.2 (CI): now also D13.5 (CO); no longer D15.4 (DIN)
- net at D30.2 (CI): now also D29.5 (CO)
- net at D18.2 (CI): now also D17.5 (CO); no longer D19.4 (DIN)
- net at D17.2 (CI): now also D16.5 (CO); no longer D18.4 (DIN)
- net at D19.2 (CI): now also D18.5 (CO); no longer D20.4 (DIN)
- net at D22.2 (CI): now also D21.5 (CO); no longer D23.4 (DIN)
- net at D23.2 (CI): now also D22.5 (CO); no longer D24.4 (DIN)
- new net: D26.6 (DO), D27.1 (DI)
- new net: D27.6 (DO), D28.1 (DI)
- new net: D15.6 (DO), D16.1 (DI)
- new net: D16.6 (DO), D17.1 (DI)
- new net: D24.6 (DO), D25.1 (DI)
- new net: D25.6 (DO), D26.1 (DI)
- new net: D28.6 (DO), D29.1 (DI)
- new net: D29.6 (DO), D30.1 (DI)
- new net: D20.6 (DO), D21.1 (DI)
- new net: D21.6 (DO), D22.1 (DI)
- new net: D13.1 (DI), IC3.4 (Y)
- new net: D13.6 (DO), D14.1 (DI)
- new net: D14.6 (DO), D15.1 (DI)
- new net: D17.6 (DO), D18.1 (DI)
- new net: D18.6 (DO), D19.1 (DI)
- new net: D19.6 (DO), D20.1 (DI)
- new net: D22.6 (DO), D23.1 (DI)
- new net: D23.6 (DO), D24.1 (DI)
- new net WLED_CLK: IC2.2 (A)
- no-connect marks 1 -> 2
Other:
- note added: "SK9B22 AKA APA102 RGB LEDs"
- note removed: "WS2812B RGB LEDs"
- moved on the sheet: IC2
