File: Hardware/Dash/AdvDash_5_inch/rtc.kicad_sch (KiCad schematic)
At the start: 7 parts, among them IC1 RV-8803-C7

Commit message: PCB R0.1.0
Other:
- company: (none) -> ADV.ECU - GNVPerformance
- title: (none) -> Real Time Clock

Commit message: :adhesive_bandage: Minor change to the PCB
Parts:
- BT1: LCSC (none) -> C70377
- C26: LCSC (none) -> C83170
- D10: LCSC (none) -> C5189799
- IC1: LCSC (none) -> C2846926
- R28, R29, R30: LCSC (none) -> C149504
Changed lines of the file:
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@@
+      (effects (font (size 1.27 1.27)) hide)
+    )
+    (property "LCSC" "C149504" (at 93.345 69.215 0)
       (effects (font (size 1.27 1.27)) hide)
     )
@@
       (effects (font (size 1.27 1.27)) hide)
     )
+    (property "LCSC" "C83170" (at 86.995 69.215 0)
+      (effects (font (size 1.27 1.27)) hide)
+    )
     (pin "1")
     (pin "2")
@@
     )
     (property "Datasheet" "~" (at 144.145 50.165 0)
+      (effects (font (size 1.27 1.27)) hide)
+    )
+    (property "LCSC" "C149504" (at 144.145 50.165 0)
       (effects (font (size 1.27 1.27)) hide)
     )
@@
     (property "Manufacturer_Part_Number" "RV-8803-C7-32.768k-3PPM-TA-QA" (at 125.73 850.165 0)
       (effects (font (size 1.27 1.27)) (justify left top) hide)
+    )
+    (property "LCSC" "C2846926" (at 99.06 55.245 0)
+      (effects (font (size 1.27 1.27)) hide)
     )
     (pin "1")
@@
       (effects (font (size 1.27 1.27)) hide)
     )
+    (property "LCSC" "C5189799" (at 83.185 52.705 0)
+      (effects (font (size 1.27 1.27)) hide)
+    )
     (pin "1")
     (pin "2")
@@
       (effects (font (size 1.27 1.27)) hide)
     )
+    (property "LCSC" "C149504" (at 140.335 50.165 0)
+      (effects (font (size 1.27 1.27)) hide)
+    )
     (pin "1")
     (pin "2")
@@
       (effects (font (size 1.27 1.27)) (justify bottom) hide)
     )
+    (property "LCSC" "C70377" (at 63.5 45.085 0)
+      (effects (font (size 1.27 1.27)) hide)
+    )
     (pin "N")
