File: Hardware/Dash/AdvDash_5_inch/usbc.kicad_sch (KiCad schematic)
At the start: 4 parts, among them J2 USB4110-GF-A, U6 USBLC6-2P6

Commit message: PCB R0.1.0
Other:
- company: (none) -> ADV.ECU - GNVPerformance
- title: (none) -> USB-C Connector

Commit message: :adhesive_bandage: Minor change to the PCB
Parts:
- R12, R15: LCSC (none) -> C84375
- U6: LCSC (none) -> C7519
Changed lines of the file:
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@@
+      (effects (font (size 1.27 1.27)) hide)
+    )
+    (property "LCSC" "C84375" (at 99.06 78.105 0)
       (effects (font (size 1.27 1.27)) hide)
     )
@@
       (effects (font (size 1.27 1.27)) hide)
     )
+    (property "LCSC" "C7519" (at 181.61 85.725 0)
+      (effects (font (size 1.27 1.27)) hide)
+    )
     (pin "1")
     (pin "2")
@@
       (effects (font (size 1.27 1.27)) hide)
     )
+    (property "LCSC" "C84375" (at 147.32 94.615 0)
+      (effects (font (size 1.27 1.27)) hide)
+    )
